File: HARDWARE/mainboard/fduino.sch (EAGLE design)
At the start: 65 parts, among them IC1 DRV8834SMD, IC2 LF50, IC3 LSM303DLHC, IC4 LSM303DLHC, Q1 CSM-7X-DU, SW1 SWITCHTHT, T1 BPX81, T2 BPX81, T3 BPX81, T4 BPX81, T5 BPX81, T6 BPX81

Commit message: common
Parts:
- removed C10, C14: 4.7u, rcl:C-EUC0603
- removed C11, C15: 10u, rcl:CPOL-EUSMCZ
- removed C12, C16, C8: 100n, rcl:C-EUC0603
- removed C13, C17: 0.22u, rcl:C-EUC0603
- removed C5: 10n, rcl:C-EUC0603
- removed IC4: LSM303DLHC, st-microelectronics:LSM303DLHC
- removed JP1: (no value), pinhead:PINHD-2X3
- removed JP2, JP3, JP4, JP5: (no value), pinhead:PINHD-1X2
- removed LED10: Orange, led:LEDSML0603
- removed MCU1: ATMEGA328PMA, martinmake:ATMEGA328PMA
- removed R17, R18, R19: 220, rcl:R-EU_R0603
- added JP-ICSP: (no value), pinhead:PINHD-2X3
- added JP-LE, JP-RE: (no value), pinhead:PINHD-1X5
- added JP-LM, JP-RM: (no value), pinhead:PINHD-1X2
- added JP-USS: (no value), pinhead:PINHD-1X4
- added LED11, LED12: White, led:LEDSML1206
- added R21, R23, R28, R30, R32: 1k, rcl:R-EU_R1206
- added R22, R24, R29, R31: 220, rcl:R-EU_R1206
- added SW2, SW3, SW4: SWITCHTHT, martinmake:SWITCHTHT
- added T7, T8: BPX81, opto-trans-siemens:BPX81
- added U$2, U$3: BAT, martinmake:BAT
- C1, C2, C3, C9: device rcl:C-EUC0603 -> rcl:C-EUC1206
- C4: value 10n -> 100u; device rcl:C-EUC0603 -> rcl:CPOL-EUSMCD
- C6: value 2.2u -> 100n; device rcl:C-EUC0603 -> rcl:C-EUC1206
- C7: value 10u -> 100n; device rcl:CPOL-EUSMCZ -> rcl:C-EUC1206
- IC1: value DRV8834SMD -> ATMEGA328PMA; device martinmake:DRV8834SMD -> martinmake:ATMEGA328PMA
- IC3: value LSM303DLHC -> L6205; device st-microelectronics:LSM303DLHC -> martinmake:L6205
- LED1, LED2, LED4, LED6, LED7, LED8, LED9: device led:LEDSML0603 -> led:LEDSML1206
- LED3: value Blue -> White; device led:LEDSML0603 -> led:LEDSML1206
- LED5: value White -> Orange; device led:LEDSML0603 -> led:LEDSML1206
- R1: value 100k -> 120; device rcl:R-EU_R0603 -> rcl:R-EU_R1206
- R10, R13, R9: value 0 -> 1k; device rcl:R-EU_R0603 -> rcl:R-EU_R1206
- R11, R16: value 220 -> 1k; device rcl:R-EU_R0603 -> rcl:R-EU_R1206
- R12: value 47k -> 220; device rcl:R-EU_R0603 -> rcl:R-EU_R1206
- R14: value 0 -> 220; device rcl:R-EU_R0603 -> rcl:R-EU_R1206
- R15, R20, R4: device rcl:R-EU_R0603 -> rcl:R-EU_R1206
- R2, R3: value 680 -> 120; device rcl:R-EU_R0603 -> rcl:R-EU_R1206
- R5, R6: value 120 -> 680; device rcl:R-EU_R0603 -> rcl:R-EU_R1206
- R7: value 120 -> 100k; device rcl:R-EU_R0603 -> rcl:R-EU_R1206
- R8: value 680 -> 220; device rcl:R-EU_R0603 -> rcl:R-EU_R1206
Connections:
- removed net N$11: IC1.AVREF, IC1.BVREF, IC1.VREFO
- removed net N$16: IC1.ADECAY, R9.1
- removed net N$17: IC1.BDECAY, R10.1
- removed net N$18: IC1.!SLEEP, R12.1
- removed net N$19: IC1.AISEN, R13.2
- removed net N$2: C13.2, IC4.SETP
- removed net N$20: R10.2, R12.2, R9.2
- removed net N$21: IC1.BISEN, R14.2
- removed net N$32 (its old number): R11.1
- removed net SCL: IC3.SLC, IC4.SLC, MCU1.PC5
- removed net SDA: IC3.SDA, IC4.SDA, MCU1.PC4
- new net ADC4: IC1.PC4, R23.2, T5.C
- new net ADC5: IC1.PC5, R28.2, T6.C
- new net ECHO: JP-USS.3
- new net GND2: LED11.C, LED12.C, LED3.C, LED4.C, LED6.C, LED7.C, LED8.C, LED9.C, T1.E, T2.E, T3.E, T4.E, T5.E, T6.E, T7.E, T8.E
- new net INT0: IC1.PD2
- new net INT1: IC1.PD3
- new net N$24: R20.1
- new net N$34: JP-LE.1
- new net N$39: JP-RE.3
- new net N$42: R11.1, R13.1, R16.1, R21.1, R23.1, R28.1, R30.1, R32.1
- new net N$43: LED4.A, R12.2
- new net N$44: JP-RE.2
- new net N$45: R8.1
- new net N$46: JP-RE.5
- new net N$47: LED3.A, R8.2
- new net N$48: JP-RE.4
- new net N$49: JP-ICSP.3, R2.1
- new net N$50: JP-ICSP.5, R1.1
- new net N$51: JP-ICSP.4, R4.1
- new net SW1: IC1.PD4, R9.1, SW2.1
- new net SW2: IC1.PD7, R10.1, SW3.1
- new net TRIG: JP-USS.2
- net !RESET: now also IC1.PC6, R7.2; no longer JP1.5, MCU1.PC6, R5.1, R5.2
- net !SS: now also IC1.PB2; no longer MCU1.PB2
- net ADC0: now also IC1.PC0, R11.2, T1.C; no longer MCU1.PC0, T1.E
- net ADC1: now also IC1.PC1, R13.2, T2.C; no longer MCU1.PC1, T2.E
- net ADC2: now also IC1.PC2, R16.2, T3.C; no longer MCU1.PC2, T3.E
- net ADC3: now also IC1.PC3, R21.2, T4.C; no longer MCU1.PC3, T4.E
- net ADC6: now also IC1.ADC6, R30.2, T7.C; no longer MCU1.ADC6, T5.E
- net ADC7: now also IC1.ADC7, R32.2, T8.C; no longer MCU1.ADC7, T6.E
- net DIRA: now also IC1.PD0, IC3.IN2A; no longer IC1.APHASE, MCU1.PD0
- net DIRB: now also IC1.PD1, IC3.IN2B; no longer IC1.BPHASE, MCU1.PD1
- net GND: now also C4.-, C7.2, IC3.SENSEA, IC3.SENSEB, JP-ICSP.6, JP-USS.4, R10.2, R9.2, U$3A.-; no longer C10.2, C11.-, C12.1, C14.2, C15.-, C16.1, C5.2, C7.-, C8.2, IC1.CONFIG, IC1.M1, IC3.RSVD@1, IC3.RSVD@2, IC4.GND, IC4.RSVD@1, IC4.RSVD@2, JP1.6, JP2.2, LED10.C, LED4.C, LED6.C, LED7.C, LED8.C, LED9.C, MCU1.GND, R13.1, R14.1
- net MISO: now also IC1.PB4, R3.2; no longer JP1.1, MCU1.PB4, R7.1, R7.2
- net MOSI: now also IC1.PB3; no longer JP1.4, MCU1.PB3, R4.1
- net N$1: now also LED6.A, R15.2; no longer C10.1, IC4.C1
- net N$10: now also U$2A.+, U$2B.-; no longer IC1.!FAULT, LED3.C
- net N$12: now also LED7.A, R20.2; no longer C13.1, IC4.SETC
- net N$13: now also JP-LE.5; no longer C14.1, IC3.C1
- net N$14: now also SW4.2, U$2B.+; no longer C4.2, IC1.VCP
- net N$15: now also U$2A.-, U$3B.+; no longer C6.1, IC1.VINT
- net N$22: now also LED12.A, R31.2; no longer LED4.A, R11.2
- net N$23: now also LED8.A, R22.2; no longer LED5.A, R15.2
- net N$26: now also JP-LE.4; no longer JP5.2, T1.C, T2.C, T3.C, T4.C, T5.C, T6.C
- net N$27: now also LED9.A, R24.2; no longer LED6.A, R16.2
- net N$28: now also R22.1; no longer R16.1
- net N$29: now also JP-LE.3; no longer C17.2, IC3.SETP
- net N$3: now also IC3.OUT2B, JP-RM.2; no longer IC1.BOUT2, JP4.2
- net N$30: now also LED11.A, R29.2; no longer C17.1, IC3.SETC
- net N$31: now also JP-LE.2; no longer LED7.A, R17.2
- net N$33: now also JP-ICSP.1, R3.1; no longer JP5.1
- net N$35: now also R24.1; no longer R17.1
- net N$36: now also LED5.A, R14.2; no longer LED10.A, R20.2
- net N$37: now also JP-RE.1; no longer LED8.A, R18.2
- net N$38: now also R29.1; no longer R18.1
- net N$4: now also R6.1; no longer R3.1
- net N$40: now also R12.1; no longer LED9.A, R19.2
- net N$41: now also R31.1; no longer R19.1
- net N$5: now also R5.1; no longer R2.1
- net N$6: now also IC3.OUT1B, JP-RM.1; no longer IC1.BOUT1, JP4.1
- net N$7: now also IC3.OUT1A, JP-LM.1; no longer IC1.AOUT1, JP3.1
- net N$8: now also IC3.OUT2A, JP-LM.2; no longer IC1.AOUT2, JP3.2
- net N$9: now also U$3A.+, U$3B.-; no longer LED3.A, R8.1
- net OC0A: now also IC1.PD6, IC3.IN1A; no longer IC1.AENBL, MCU1.PD6
- net OC0B: now also IC1.PD5, IC3.IN1B; no longer IC1.BENBL, MCU1.PD5
- net PB0: now also IC1.PB0; no longer MCU1.PB0
- net PB1: now also IC1.PB1; no longer MCU1.PB1
- net SCK: now also IC1.PB5, R2.2; no longer JP1.3, MCU1.PB5, R6.1, R6.2
- net VCC: now also IC1.AREF, IC1.AVCC, IC1.VCC, IC3.ENA, IC3.ENB, IC3.VBOOT, IC3.VCP, JP-ICSP.2, JP-USS.1, R14.1, R5.2, R6.2, R7.1, SW2.2, SW3.2; no longer C11.+, C12.2, C15.+, C16.2, IC3.VDD, IC3.VDD_IO, IC4.VDD, IC4.VDD_IO, JP1.2, JP2.1, MCU1.AREF, MCU1.AVCC, MCU1.VCC, R1.1, R2.2, R20.1, R3.2, R8.2
- net VM: now also C4.+, C6.1, C7.1, IC3.VSA, IC3.VSB, SW4.1; no longer C4.1, C5.1, C7.+, C8.1, IC1.VM
- net XTAL1: now also IC1.PB6; no longer MCU1.PB6
- net XTAL2: now also IC1.PB7; no longer MCU1.PB7
Other:
- note added: "Martin Michalec"
- moved on the sheet: C1, C2, C3, C6, C9, IC2, LED1, LED2, LED3, LED4, LED5, LED6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
