File: HARDWARE/mainboard/FDUINO.brd (EAGLE design)
At the start: 150 x 90 mm, 68 parts, among them IC1 ATMEGA328PMA, IC2 LF50, IC3 L6205, Q1 CSM-7X-DU, SW1 SWITCHTHT, SW2 SWITCHTHT, SW3 SWITCHTHT, SW4 SWITCHTHT, T1 BPX81, T2 BPX81, T3 BPX81, T4 BPX81, T5 BPX81, T6 BPX81, T7 BPX81, T8 BPX81

Commit message: added UART connector, USR button, motor connectors, charge pump for motor driver
Parts:
- removed JP-LE, JP-RE: (no value), pinhead:1X05
- removed JP-LM, JP-RM: (no value), pinhead:1X02
- removed LED11: White, led:SML1206
- removed R28, R30: 1k, rcl:R1206
- removed R29, R31: 220, rcl:R1206
- removed SW3: SWITCHTHT, martinmake:SWITCH
- removed U$2, U$3: BAT, martinmake:BAT2X18650
- added BAT1, BAT2: BATSERIES, martinmake:BAT2X18650SERIES
- added C5, C8: 100n, rcl:C1206
- added D1, D2: 1N4148, diode:DO35-7
- added JP3: UART, pinhead:1X06/90
- added R17, R18: 220, rcl:R1206
- added R19: 10k, rcl:R1206
- added ZH1: LM, jst:B5B-ZR
- added ZH2: RM, jst:B5B-ZR
- C7, C9: value 100n -> 10n
- JP1: value (none) -> ICSP
- JP2: value (none) -> USS
- LED2: value Purple -> White
- LED4: value White -> Orange
- LED5: value Orange -> White
- R10, R13: value 1k -> 220
- R11, R16, R21, R23, R25, R9: value 1k -> 10k
- R14: value 220 -> 10k
- R5: value 680 -> 1k
- moved C9 224.1 mm to (2.54, -144.8), turned to 0 degrees
- moved C7 181.9 mm to (2.54, -119.4), turned to 0 degrees
- moved R9 70.8 mm to (21.6, 36.8), flipped to the bottom, turned to 90 degrees
- moved R10 53.5 mm to (14.0, 47.0), flipped to the bottom, turned to 90 degrees
- moved LED2 53.4 mm to (16.5, 36.8), flipped to the bottom, turned to 90 degrees
- moved LED9 50.6 mm to (10.2, 10.2)
- moved LED5 45.0 mm to (16.5, 55.9), flipped to the bottom, turned to 90 degrees
- moved R23 42.7 mm to (15.2, 10.2)
- moved R22 42.5 mm to (7.62, 10.4)
- moved R5 41.8 mm to (87.6, 11.4), turned to 180 degrees
- moved LED4 39.9 mm to (50.8, 26.7), flipped to the top, turned to 180 degrees
- moved R12 38.8 mm to (49.5, 31.5), flipped to the top, turned to 270 degrees
- moved R14 37.1 mm to (21.6, 55.9), flipped to the bottom, turned to 90 degrees
- moved R24 32.4 mm to (7.62, 80.2)
- moved C6 31.4 mm to (106.7, 45.6), turned to 90 degrees
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- renumbered JP-ICSP to JP1, JP-USS to JP2, LED12 to LED10, R32 to R25, SW1 to S2, SW2 to USR, SW4 to S3
Connections:
- net PB0 renamed LED
- removed net N$12 (its old number): LED7.A, R20.2
- removed net N$13: JP-LE.5
- removed net N$26: JP-LE.4
- removed net N$29: JP-LE.3
- removed net N$31: JP-LE.2
- removed net N$34: JP-LE.1
- removed net N$36 (its old number): LED5.A, R14.2
- removed net N$37: JP-RE.1
- removed net N$38 (its old number): R29.1
- removed net N$39: JP-RE.3
- removed net N$41 (its old number): R31.1
- removed net N$42: R11.1, R13.1, R16.1, R21.1, R23.1, R25.1, R28.1, R30.1
- removed net N$44: JP-RE.2
- removed net N$46: JP-RE.5
- removed net N$48: JP-RE.4
- removed net N$6: IC3.7, JP-RM.1
- removed net N$8: IC3.18, JP-LM.2
- removed net PB1: IC1.13, LED2.C
- removed net SW1: IC1.2, R9.1, USR.P$1
- removed net SW2: IC1.11, R10.1, SW3.P$1
- new net N$1: LED5.A, R13.2
- new net N$2: C9.1, D2.C, IC3.12
- new net N$28: R18.1
- new net N$32: R13.1
- new net N$43: LED3.A, R10.2
- new net OUT1A: IC3.4, ZH1.1
- new net OUT1B: IC3.7, ZH2.1
- new net OUT2A: IC3.18, ZH1.5
- new net OUT2B: IC3.13, ZH2.5
- new net RX: IC1.30, JP3.4
- new net TX: IC1.31, JP3.5
- new net USR: IC1.13, R5.1, USR.P$1
- net ADC0: now also R9.2; no longer R11.2
- net ADC1: now also R11.2; no longer R13.2
- net ADC2: now also R14.2; no longer R16.2
- net ADC3: now also R16.2; no longer R21.2
- net ADC4: now also R19.2; no longer R23.2
- net ADC5: now also R21.2; no longer R28.2
- net ADC6: now also R23.2; no longer R30.2
- net DIRA: now also IC1.2; no longer IC1.30
- net DIRB: now also IC1.11; no longer IC1.31
- net GND: now also BAT2.-@1, C5.2, C8.2, JP3.1, LED4.C, R5.2, ZH1.3, ZH2.3; no longer C7.2, C9.2, LED5.C, R10.2, R9.2, U$3.-@1
- net GND2: now also LED2.C, LED5.C; no longer LED11.C, LED4.C
- net INT0: now also ZH1.2
- net INT1: now also ZH2.2
- net N$10: now also BAT1.+@1, BAT1.-@2; no longer U$2.+@1, U$2.-@2
- net N$14: now also BAT1.+@2; no longer U$2.+@2
- net N$15: now also BAT1.-@1, BAT2.+@2; no longer U$2.-@1, U$3.+@2
- net N$22: now also R24.2; no longer R31.2
- net N$23: now also LED7.A, R18.2; no longer LED8.A, R22.2
- net N$27: now also LED8.A, R20.2; no longer LED9.A, R24.2
- net N$3: now also D1.C, D2.A, R17.2; no longer IC3.13, JP-RM.2
- net N$30: now also LED9.A, R22.2; no longer LED11.A, R29.2
- net N$4: now also C7.2, R17.1; no longer LED2.A, R6.1
- net N$40: now also R10.1; no longer R12.1
- net N$47: now also LED2.A; no longer LED3.A
- net N$5: now also R6.1; no longer R5.1
- net N$7: now also C7.1, IC3.19; no longer IC3.4, JP-LM.1
- net N$9: now also BAT2.+@1, BAT2.-@2; no longer U$3.+@1, U$3.-@2
- net VCC: now also C8.1, JP3.3, R11.1, R12.1, R16.1, R19.1, R21.1, R23.1, R25.1, R9.1, ZH1.4, ZH2.4; no longer C9.1, IC3.12, IC3.19, R5.2, SW3.P$2
- net VM: now also C5.1, C9.2, D1.A; no longer C7.1
Routing:
- net OC0A: track 0.00 -> 32.0 mm
- net XTAL2: track 5.76 -> 18.3 mm
- net XTAL1: track 5.61 -> 17.5 mm
- net PB1: track 7.62 -> 0.00 mm
- net USR: track 0.00 -> 6.26 mm
- net VM: track 7.82 -> 12.1 mm
- net N$36 (its old number): track 3.52 -> 0.00 mm
- net N$4: track 3.18 -> 0.00 mm
- net SW2: track 2.91 -> 0.00 mm
- net N$43: track 0.00 -> 2.68 mm
- net N$1: track 0.00 -> 2.68 mm
- net N$12 (its old number): track 2.68 -> 0.00 mm
- net VCC: track 8.08 -> 10.1 mm
- net N$36: track 2.68 -> 3.52 mm
