File: HARDWARE/mainboard/mainboard.brd (EAGLE design)
At the start: 150 x 90 mm, 68 parts, among them IC1 ATMEGA328PMA, IC2 LF50, IC3 L6205, Q1 CSM-7X-DU, T1 BPX81, T2 BPX81, T3 BPX81, T4 BPX81, T5 BPX81, T6 BPX81, T7 BPX81, T8 BPX81

Commit message: added gyroscope and distance sensors
Parts:
- removed LED7, LED8: White, led:SML1206
- removed R18, R20: 220, rcl:R1206
- removed R19, R21: 10k, rcl:R1206
- removed T5, T6: BPX81, opto-trans-siemens:BPX81
- added C10: 10n, rcl:C1206
- added C11, C12: 100n, rcl:C1206
- added C13: 10u, rcl:SMC_D
- added IC4: L3GD20HSMD, martinmake:LGA-16
- added JP4: LDS, pinhead:1X04/90
- added JP5: FDS, pinhead:1X04/90
- JP2: value USS -> RDS; device pinhead:1X04 -> pinhead:1X04/90
- moved ZH1 231.9 mm to (144.8, 87.6), turned to 90 degrees
- moved JP3 217.2 mm to (149.9, 55.9), turned to 270 degrees
- moved D2 200.6 mm to (110.5, 33.0), turned to 90 degrees
- moved C9 200.2 mm to (108.0, 25.4), turned to 180 degrees
- moved D1 192.5 mm to (105.4, 33.0), turned to 270 degrees
- moved R17 190.4 mm to (101.6, 36.8)
- moved C7 188.2 mm to (101.6, 40.6), turned to 180 degrees
- moved ZH2 180.2 mm to (146.1, 22.9), turned to 90 degrees
- moved JP2 102.6 mm to (87.6, 108.0), turned to 0 degrees
- moved R5 95.2 mm to (118.1, 101.6), turned to 90 degrees
- moved USR 94.0 mm to (121.9, 101.6), turned to 270 degrees
- moved LED9 70.0 mm to (15.2, 80.0)
- moved R22 70.0 mm to (12.7, 80.2)
- moved R23 70.0 mm to (20.3, 80.0)
- moved T7 70.0 mm to (17.8, 80.0), flipped to the bottom
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Connections:
- removed net ADC4: IC1.27, R19.2, T5.C
- removed net ADC5: IC1.28, R21.2, T6.C
- removed net ECHO: JP2.3
- removed net N$23: LED7.A, R18.2
- removed net N$27: LED8.A, R20.2
- removed net N$28: R18.1
- removed net N$35: R20.1
- removed net TRIG: JP2.2
- new net N$11: IC4.6
- new net N$13: IC4.7
- new net N$6: C10.1, IC4.14
- new net SCL: IC1.28, IC4.2, JP2.3, JP4.4, JP5.4
- new net SDA: IC1.27, IC4.3, JP2.4, JP4.3, JP5.3
- net GND: now also C10.2, C11.2, C12.2, C13.-, IC4.10, IC4.11, IC4.12, IC4.13, IC4.15, IC4.9, JP2.2, JP4.2, JP5.2; no longer JP2.4
- net GND2: no longer LED7.C, LED8.C, T5.E, T6.E
- net VCC: now also C11.1, C12.1, C13.+, IC4.1, IC4.16, IC4.4, IC4.5, IC4.8, JP4.1, JP5.1; no longer R19.1, R21.1
Routing:
- net GND: track 77.9 -> 102.3 mm, vias 1 -> 3
- net VCC: track 10.1 -> 33.8 mm
- net N$7: track 0.00 -> 20.4 mm, vias 0 -> 2
- net !RESET: track 31.6 -> 48.9 mm, vias 0 -> 1
- net OC0A: track 32.0 -> 19.3 mm
- net N$3: track 0.00 -> 7.47 mm
- net GND2: track 21.9 -> 16.4 mm
- net N$6: track 0.00 -> 4.27 mm
- net N$2: track 0.00 -> 3.98 mm
- net N$4: track 0.00 -> 3.82 mm
- net TX: track 0.00 -> 3.16 mm, vias 0 -> 1
- net N$23: track 2.68 -> 0.00 mm
- net ADC5: track 2.60 -> 0.00 mm
- net ADC4: track 2.60 -> 0.00 mm
- net N$27: track 2.58 -> 0.00 mm
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Other:
- board size 150 x 90 mm -> 150 x 110.3 mm
