File: HARDWARE/mainboard/mainboard.sch (EAGLE design)
At the start: 68 parts, among them IC1 ATMEGA328PMA, IC2 LF50, IC3 L6205, Q1 CSM-7X-DU, T1 BPX81, T2 BPX81, T3 BPX81, T4 BPX81, T5 BPX81, T6 BPX81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

Commit message: added gyroscope and distance sensors
Parts:
- removed LED7, LED8: White, led:LEDSML1206
- removed R18, R20: 220, rcl:R-EU_R1206
- removed R19, R21: 10k, rcl:R-EU_R1206
- removed T5, T6: BPX81, opto-trans-siemens:BPX81
- added C10: 10n, rcl:C-EUC1206
- added C11, C12: 100n, rcl:C-EUC1206
- added C13: 10u, rcl:CPOL-EUSMCD
- added IC4: L3GD20HSMD, martinmake:L3GD20HSMD
- added JP4: LDS, pinhead:PINHD-1X4/90
- added JP5: FDS, pinhead:PINHD-1X4/90
- JP2: value USS -> RDS; device pinhead:PINHD-1X4 -> pinhead:PINHD-1X4/90
Connections:
- removed net ADC4: IC1.PC4, R19.2, T5.C
- removed net ADC5: IC1.PC5, R21.2, T6.C
- removed net ECHO: JP2.3
- removed net N$23: LED7.A, R18.2
- removed net N$27: LED8.A, R20.2
- removed net N$28: R18.1
- removed net N$35: R20.1
- removed net TRIG: JP2.2
- new net N$11: IC4.DRDY/INT2
- new net N$13: IC4.INT1
- new net N$6: C10.1, IC4.CAP
- new net SCL: IC1.PC5, IC4.SCL/SPC, JP2.3, JP4.4, JP5.4
- new net SDA: IC1.PC4, IC4.SDA/SDI/SDO, JP2.4, JP4.3, JP5.3
- net GND: now also C10.2, C11.2, C12.2, C13.-, IC4.GND, JP2.2, JP4.2, JP5.2; no longer JP2.4
- net GND2: no longer LED7.C, LED8.C, T5.E, T6.E
- net VCC: now also C11.1, C12.1, C13.+, IC4.CS, IC4.DEN, IC4.SA0/SDO, IC4.VDD, IC4.VDD_IO, JP4.1, JP5.1; no longer R19.1, R21.1
Other:
- note added: "Gyro Sensor"
- note added: "Laser Distance Sensors"
- note removed: "Ultra Sonic Sensor"
- moved on the sheet: C4, C6, C7, C9, D1, D2, IC1, IC3, JP1, JP2, LED1, LED2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
