File: HARDWARE/line_follower/line_follower.brd (EAGLE design)
At the start: 85.4 x 88.9 mm, 74 parts, among them IC1 L3GD20HSMD, IC2 L6205, IC3 ATMEGA328PMA, IC4 LF33, J1 FFC2B05-10-X_REVC, J2 FFC2B05-10-X_REVC, Q1 10MHz, T1 ELPT15-21C, T2 ELPT15-21C, T3 ELPT15-21C, T4 ELPT15-21C, T5 ELPT15-21C, T6 ELPT15-21C, X1 MINI-USB-SCHIELD-32005-301

Commit message: common
Parts:
- removed ZH1: LM, jst:B5B-ZR
- removed ZH2: RM, jst:B5B-ZR
- added PH1: LM, SparkFun-Connectors:JST-5-PTH-VERT
- added PH2: RM, SparkFun-Connectors:JST-5-PTH-VERT
- moved JP7 32.7 mm to (62.2, 35.6), turned to 180 degrees
- moved R1 6.79 mm to (83.2, 74.9), turned to 90 degrees
- moved R2 6.68 mm to (83.2, 68.6), turned to 270 degrees
- moved LED2 1.29 mm to (76.2, 69.8)
- moved S2 1.27 mm to (77.8, 21.6)
- moved LED1 0.31 mm to (76.2, 73.7)
- moved R19 0.27 mm to (40.0, 9.14)
Connections:
- net GND: now also PH1.3, PH2.3; no longer ZH1.3, ZH2.3
- net INT0: now also PH1.2; no longer ZH1.2
- net INT1: now also PH2.2; no longer ZH2.2
- net OUT1A: now also PH1.1; no longer ZH1.1
- net OUT1B: now also PH2.1; no longer ZH2.1
- net OUT2A: now also PH1.5; no longer ZH1.5
- net OUT2B: now also PH2.5; no longer ZH2.5
- net VCC: now also PH1.4, PH2.4; no longer ZH1.4, ZH2.4
Routing:
- net GND: track 119.1 -> 83.8 mm
- net F_VCC: track 30.2 -> 34.6 mm
- net VB: track 74.3 -> 71.1 mm
- net N$13: track 2.68 -> 5.30 mm
- net N$5: track 2.68 -> 5.30 mm
- net OUT1B: track 53.1 -> 54.6 mm
- net TX: track 25.7 -> 26.7 mm
- net RX: track 29.5 -> 30.5 mm
- net N$10: track 35.4 -> 34.5 mm
- net OUT2A: track 49.7 -> 50.6 mm
- net OUT2B: track 41.9 -> 42.8 mm
- net INT1: track 64.4 -> 65.2 mm
- net LEDA: track 44.7 -> 43.9 mm
- net VUSB: track 32.5 -> 32.0 mm
Other:
- outline, holes or cut-outs redrawn

Commit message: common
Parts:
- moved JP1 0.71 mm to (29.2, 75.6)
- moved R1 0.64 mm to (82.5, 74.9)
- moved R2 0.64 mm to (82.5, 68.6)
- moved R19 0.63 mm to (39.4, 9.05)
- moved C4 0.63 mm to (34.9, 73.7)
- moved R16 0.63 mm to (35.6, 17.8)
- moved R17 0.63 mm to (38.1, 17.8)
- moved R18 0.63 mm to (40.6, 17.8)
- moved IC1 0.63 mm to (29.2, 69.8)
- moved JP6 0.63 mm to (38.1, 12.7)
- moved C1 0.45 mm to (39.4, 78.1)
- moved S3 0.39 mm to (36.2, 61.0)
- moved C16 0.35 mm to (34.3, 62.2)
- moved PH2 0.33 mm to (78.1, 82.5)
- moved PH1 0.33 mm to (78.1, 6.35)
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Routing:
- net SCL: track 100.4 -> 101.2 mm
- net N$5: track 5.30 -> 4.66 mm
- net N$13: track 5.30 -> 4.66 mm
- net GND: track 83.8 -> 84.4 mm
Other:
- board size 85.4 x 88.9 mm -> 85.1 x 88.9 mm
- board text removed: "/home/arch/Documents/proj/slate_vixen/HARDWARE/line_follower/printing/dragon_head.bmp"
