File: HARDWARE/line_follower/line_follower.sch (EAGLE design)
At the start: 67 parts, among them IC1 ATMEGA328PMA, IC2 LF50, IC3 L6205, IC4 L3GD20HSMD, Q1 CSM-7X-DU, T1 BPX81, T2 BPX81, T3 BPX81, T4 BPX81, T7 BPX81, T8 BPX81

Commit message: finished front module
Parts:
- removed BAT1, BAT2: BATSERIES, martinmake:BATSERIES
- removed LED9: White, led:LEDSML1206
- removed R22, R24: 220, rcl:R-EU_R1206
- removed R23, R25: 10k, rcl:R-EU_R1206
- removed T7, T8: BPX81, opto-trans-siemens:BPX81
- removed USR: SWITCHTHT, martinmake:SWITCHTHT
- added J1, J2: FFC2B05-10-X_REVC, FFC2B05-10-X_REVC:FFC2B05-10-X_REVC
- added JP6: ICSP, pinhead:PINHD-2X3
- added JP7: 3S/4S, pinhead:PINHD-1X2
- added LED8: Orange, led:LEDSML1206
- added R18, R19: 120, rcl:R-EU_R1206
- added R20: 220, rcl:R-EU_R1206
- added R21: 100k, rcl:R-EU_R1206
- added S1: BUTTON, martinmake:BUTTON
- added T5, T6: ELPT15-21C, martinmake:ELPT15-21C
- added X1: MINI-USB-SCHIELD-32005-201, con-cypressindustries:MINI-USB-SCHIELD-32005-201
- C1: value 22p -> 10u; device rcl:C-EUC1206 -> rcl:CPOL-EUSMCD
- C10, C9: value 10n -> 22p
- C13: value 10u -> 100n; device rcl:CPOL-EUSMCD -> rcl:C-EUC1206
- C2: value 22p -> 100n
- C4: value 100u -> 10n; device rcl:CPOL-EUSMCD -> rcl:C-EUC1206
- C5: value 100n -> 100u; device rcl:C-EUC1206 -> rcl:CPOL-EUSMCD
- C8: value 100n -> 10n
- D1, D2: device diode:1N4148DO35-7 -> martinmake:DIODE
- IC1: value ATMEGA328PMA -> L3GD20HSMD; device martinmake:ATMEGA328PMA -> martinmake:L3GD20HSMD
- IC2: value LF50 -> L6205; device linear:LM340MP-05 -> martinmake:L6205
- IC3: value L6205 -> ATMEGA328PMA; device martinmake:L6205 -> martinmake:ATMEGA328PMA
- IC4: value L3GD20HSMD -> LF33; device martinmake:L3GD20HSMD -> linear:LM340MP-05
- JP1: value ICSP -> (none); device pinhead:PINHD-2X3 -> pinhead:PINHD-1X2
- JP2: value RDS -> UART; device pinhead:PINHD-1X4/90 -> pinhead:PINHD-1X6/90
- JP3: value UART -> RDS; device pinhead:PINHD-1X6/90 -> pinhead:PINHD-1X4/90
- LED4: value Orange -> White
- Q1: value CSM-7X-DU -> 10MHz
- R1: value 120 -> 680
- R13, R15: value 220 -> 10k
- R14: value 10k -> 220
- R16: value 10k -> 120
- R17: value 220 -> 120
- R2: value 120 -> 1k
- R3, R4: value 120 -> 220
- R5: value 1k -> 10k
- R6: value 680 -> 220
- R7: value 100k -> 10k
- S2: value SWITCHTHT -> DUALSWITCH; device martinmake:SWITCHTHT -> martinmake:DUALSWITCH
- S3: value SWITCHTHT -> BUTTON; device martinmake:SWITCHTHT -> martinmake:BUTTON
- T1, T2, T3, T4: value BPX81 -> ELPT15-21C; device opto-trans-siemens:BPX81 -> martinmake:ELPT15-21C
- renumbered LED10 to LED7
Connections:
- removed net GND2: LED2.C, LED3.C, LED5.C, LED6.C, LED7.C, LED9.C, T1.E, T2.E, T3.E, T4.E, T7.E, T8.E
- removed net N$10: BAT1A.+, BAT1B.-
- removed net N$11: IC4.DRDY/INT2
- removed net N$13: IC4.INT1
- removed net N$14: BAT1B.+, S3.2
- removed net N$15: BAT1A.-, BAT2B.+
- removed net N$24: R15.1
- removed net N$32: R13.1
- removed net N$38: R22.1
- removed net N$40: R10.1
- removed net N$41: R24.1
- removed net N$45: R8.1
- removed net VM: C4.+, C5.1, C6.1, C9.2, D1.A, IC2.VI, IC3.VSA, IC3.VSB, S3.1
- new net F_ADC0: J1.2, R5.2, T1.C
- new net F_ADC1: J1.3, R7.2, T2.C
- new net F_ADC2: J1.4, R9.2, T3.C
- new net F_ADC3: J1.7, R11.2, T4.C
- new net F_ADC6: J1.8, R13.2, T5.C
- new net F_ADC7: J1.9, R15.2, T6.C
- new net F_GND: J1.10, J1.SHIELD, JP5.2, LED2.C, LED3.C, LED4.C, LED5.C, LED6.C, LED7.C, T1.E, T2.E, T3.E, T4.E, T5.E, T6.E
- new net F_SCL: J1.5, JP5.4
- new net F_SDA: J1.6, JP5.3
- new net F_VCC: J1.1, JP5.1, R10.1, R11.1, R12.1, R13.1, R14.1, R15.1, R4.1, R5.1, R6.1, R7.1, R8.1, R9.1
- new net N$8: IC1.INT1, JP1.1
- new net VB: C11.1, C5.+, C6.1, C7.2, D1.A, IC2.VSA, IC2.VSB, IC4.VI, JP7.1, S2.A, S2.COM
- new net VUSB: S2.B, X1G$1.1
- net !RESET: now also C13.1, IC3.PC6, R16.2, R21.2, S3.1; no longer C3.1, IC1.PC6, R1.2, R7.2, S2.2
- net !SS: now also IC3.PB2; no longer IC1.PB2
- net ADC0: now also IC3.PC0, J2.2; no longer IC1.PC0, R9.2, T1.C
- net ADC1: now also IC3.PC1, J2.3; no longer IC1.PC1, R11.2, T2.C
- net ADC2: now also IC3.PC2, J2.4; no longer IC1.PC2, R14.2, T3.C
- net ADC3: now also IC3.PC3, J2.7; no longer IC1.PC3, R16.2, T4.C
- net ADC6: now also IC3.ADC6, J2.8; no longer IC1.ADC6, R23.2, T7.C
- net ADC7: now also IC3.ADC7, J2.9; no longer IC1.ADC7, R25.2, T8.C
- net DIRA: now also IC2.IN2A, IC3.PD4; no longer IC1.PD4, IC3.IN2A
- net DIRB: now also IC2.IN2B, IC3.PD7; no longer IC1.PD7, IC3.IN2B
- net GND: now also C1.-, C10.1, C13.2, C2.2, C4.2, C5.-, C9.1, IC2.SENSEA, IC2.SENSEB, J2.10, J2.SHIELD, JP2.1, JP3.2, JP6.6, JP7.2, LED8.C, R2.2, S3.2, X1G$1.5, X1S.S1, X1S.S2, X1S.S3, X1S.S4; no longer BAT2A.-, C1.1, C10.2, C13.-, C2.1, C4.-, C5.2, C8.2, IC3.SENSEA, IC3.SENSEB, JP1.6, JP2.2, JP3.1, JP5.2, LED4.C, R5.2, S2.1
- net INT0: now also IC3.PD2; no longer IC1.PD2
- net INT1: now also IC3.PD3; no longer IC1.PD3
- net LED: now also IC3.PB0; no longer IC1.PB0
- net MISO: now also IC3.PB4, R18.2; no longer IC1.PB4, R3.2
- net MOSI: now also IC3.PB3, R19.2; no longer IC1.PB3, R4.2
- net N$1: now also LED4.A, R8.2; no longer LED5.A, R13.2
- net N$12: now also LED5.A, R10.2; no longer LED6.A, R15.2
- net N$2: now also C7.1, IC2.VBOOT; no longer C9.1, IC3.VBOOT
- net N$22: now also R14.2; no longer R24.2
- net N$3: now also R3.2; no longer R17.2
- net N$30: now also LED6.A, R12.2; no longer LED9.A, R22.2
- net N$33: now also JP6.1, R18.1; no longer JP1.1, R3.1
- net N$36: now also LED8.A, R20.2; no longer LED4.A, R12.2
- net N$4: now also C8.2, R3.1; no longer C7.2, R17.1
- net N$43: now also R6.2; no longer R10.2
- net N$47: now also R4.2; no longer R8.2
- net N$49: now also JP6.3, R17.1; no longer JP1.3, R2.1
- net N$5: now also R1.1; no longer R6.1
- net N$50: now also JP6.5, R16.1; no longer JP1.5, R1.1
- net N$51: now also JP6.4, R19.1; no longer JP1.4, R4.1
- net N$6: now also C4.1, IC1.CAP; no longer C10.1, IC4.CAP
- net N$7: now also C8.1, IC2.VCP; no longer C7.1, IC3.VCP
- net N$9: now also IC1.DRDY/INT2, JP1.2; no longer BAT2A.+, BAT2B.-
- net OC0A: now also IC2.IN1A, IC3.PD6; no longer IC1.PD6, IC3.IN1A
- net OC0B: now also IC2.IN1B, IC3.PD5; no longer IC1.PD5, IC3.IN1B
- net OUT1A: now also IC2.OUT1A; no longer IC3.OUT1A
- net OUT1B: now also IC2.OUT1B; no longer IC3.OUT1B
- net OUT2A: now also IC2.OUT2A; no longer IC3.OUT2A
- net OUT2B: now also IC2.OUT2B; no longer IC3.OUT2B
- net RX: now also IC3.PD0, JP2.4; no longer IC1.PD0, JP3.4
- net SCK: now also IC3.PB5, R17.2; no longer IC1.PB5, R2.2
- net SCL: now also IC1.SCL/SPC, IC3.PC5, J2.5, JP3.4; no longer IC1.PC5, IC4.SCL/SPC, JP2.3, JP5.4
- net SDA: now also IC1.SDA/SDI, IC3.PC4, J2.6, JP3.3; no longer IC1.PC4, IC4.SDA/SDI/SDO, JP2.4, JP5.3
- net TX: now also IC3.PD1, JP2.5; no longer IC1.PD1, JP3.5
- net USR: now also IC3.PB1, R2.1, S1.1; no longer IC1.PB1, R5.1, USR.1
- net VCC: now also C1.+, C2.1, C3.1, IC1.CS, IC1.DEN, IC1.SA0/SDO, IC1.VDD, IC1.VDD_IO, IC2.ENA, IC2.ENB, IC3.AREF, IC3.AVCC, IC3.VCC, IC4.VO, J2.1, JP2.3, JP3.1, JP6.2, R1.2, R20.1, R21.1, S1.2; no longer C11.1, C13.+, C8.1, IC1.AREF, IC1.AVCC, IC1.VCC, IC2.VO, IC3.ENA, IC3.ENB, IC4.CS, IC4.DEN, IC4.SA0/SDO, IC4.VDD, IC4.VDD_IO, JP1.2, JP2.1, JP3.3, JP5.1, R11.1, R12.1, R14.1, R16.1, R23.1, R25.1, R6.2, R7.1, R9.1, USR.2
- net XTAL1: now also C9.2, IC3.PB6; no longer C1.2, IC1.PB6
- net XTAL2: now also C10.2, IC3.PB7; no longer C2.2, IC1.PB7
Other:
- note added: "Distance Sensors"
- note removed: "Laser Distance Sensors"

Commit message: finished PCB
Connections:
- new net N$10: C11.1, IC4.VI, S2.COM
- net VB: no longer C11.1, IC4.VI, S2.COM
Changed lines of the file:
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@@
 <attribute name="VALUE" x="-48.768" y="16.51" size="1.778" layer="96" rot="R90"/>
 </instance>
-<instance part="P+13" gate="VCC" x="-10.16" y="2.54" smashed="yes">
-<attribute name="VALUE" x="-10.16" y="3.81" size="1.778" layer="96" rot="R180" align="center"/>
+<instance part="P+13" gate="VCC" x="-12.7" y="2.54" smashed="yes">
+<attribute name="VALUE" x="-12.7" y="3.81" size="1.778" layer="96" rot="R180" align="center"/>
 </instance>
 <instance part="C13" gate="G$1" x="13.97" y="-5.08" smashed="yes" rot="MR270">
@@
 <bus name="MISO,MOSI,MOSIR,!RESET,SCK,!SS,XTAL1,XTAL2">
 <segment>
-<wire x1="-12.7" y1="17.78" x2="-12.7" y2="12.7" width="0.762" layer="92"/>
 <wire x1="-17.78" y1="22.86" x2="-12.7" y2="17.78" width="0.762" layer="92"/>
 <wire x1="-50.8" y1="22.86" x2="-17.78" y2="22.86" width="0.762" layer="92"/>
+<wire x1="-12.7" y1="17.78" x2="-12.7" y2="7.62" width="0.762" layer="92"/>
 </segment>
 <segment>
@@
 <segment>
 <pinref part="R21" gate="G$1" pin="1"/>
-<wire x1="-10.16" y1="0" x2="-10.16" y2="-2.54" width="0.1524" layer="91"/>
-<wire x1="-10.16" y1="-2.54" x2="-7.62" y2="-2.54" width="0.1524" layer="91"/>
+<wire x1="-12.7" y1="0" x2="-12.7" y2="-2.54" width="0.1524" layer="91"/>
+<wire x1="-12.7" y1="-2.54" x2="-7.62" y2="-2.54" width="0.1524" layer="91"/>
 <pinref part="P+13" gate="VCC" pin="VCC"/>
 </segment>
@@
 <net name="!RESET" class="0">
 <segment>
+<wire x1="-55.88" y1="99.06" x2="-53.34" y2="101.6" width="0.1524" layer="91"/>
+<pinref part="IC3" gate="&gt;NAME" pin="PC6"/>
+<wire x1="-53.34" y1="101.6" x2="-43.18" y2="101.6" width="0.1524" layer="91"/>
+<label x="-53.34" y="101.6" size="1.778" layer="95"/>
+</segment>
+<segment>
+<pinref part="R16" gate="G$1" pin="2"/>
+<wire x1="-50.8" y1="17.78" x2="-50.8" y2="20.32" width="0.1524" layer="91"/>
+<wire x1="-48.26" y1="22.86" x2="-50.8" y2="20.32" width="0.1524" layer="91"/>
+<label x="-34.29" y="10.16" size="1.778" layer="255" rot="MR0"/>
+</segment>
+<segment>
+<wire x1="-12.7" y1="7.62" x2="-10.16" y2="5.08" width="0.1524" layer="91"/>
+<wire x1="-10.16" y1="5.08" x2="5.08" y2="5.08" width="0.1524" layer="91"/>
 <pinref part="R21" gate="G$1" pin="2"/>
-<label x="5.08" y="3.81" size="1.778" layer="95" rot="R180" align="top-center"/>
 <wire x1="2.54" y1="-2.54" x2="5.08" y2="-2.54" width="0.1524" layer="91"/>
 <pinref part="C13" gate="G$1" pin="1"/>
-<wire x1="5.08" y1="-2.54" x2="5.08" y2="2.54" width="0.1524" layer="91"/>
 <wire x1="11.43" y1="-5.08" x2="7.62" y2="-5.08" width="0.1524" layer="91"/>
 <wire x1="7.62" y1="-5.08" x2="7.62" y2="-2.54" width="0.1524" layer="91"/>
@@
 <wire x1="7.62" y1="0" x2="10.16" y2="0" width="0.1524" layer="91"/>
 <pinref part="S3" gate="G$1" pin="1"/>
-</segment>
-<segment>
-<wire x1="-55.88" y1="99.06" x2="-53.34" y2="101.6" width="0.1524" layer="91"/>
-<pinref part="IC3" gate="&gt;NAME" pin="PC6"/>
-<wire x1="-53.34" y1="101.6" x2="-43.18" y2="101.6" width="0.1524" layer="91"/>
-<label x="-53.34" y="101.6" size="1.778" layer="95"/>
-</segment>
-<segment>
-<pinref part="R16" gate="G$1" pin="2"/>
-<wire x1="-50.8" y1="17.78" x2="-50.8" y2="20.32" width="0.1524" layer="91"/>
-<wire x1="-48.26" y1="22.86" x2="-50.8" y2="20.32" width="0.1524" layer="91"/>
-<label x="-34.29" y="10.16" size="1.778" layer="255" rot="MR0"/>
+<wire x1="5.08" y1="5.08" x2="5.08" y2="-2.54" width="0.1524" layer="91"/>
+<label x="-10.16" y="5.08" size="1.778" layer="95"/>
 </segment>
 </net>
@@
 </net>
 <net name="VB" class="0">
-<segment>
-<wire x1="58.42" y1="10.16" x2="60.96" y2="10.16" width="0.1524" layer="91"/>
-<pinref part="IC4" gate="A" pin="VI"/>
-<pinref part="C11" gate="G$1" pin="1"/>
-<wire x1="60.96" y1="10.16" x2="63.5" y2="10.16" width="0.1524" layer="91"/>
-<wire x1="60.96" y1="8.89" x2="60.96" y2="10.16" width="0.1524" layer="91"/>
-<junction x="60.96" y="10.16"/>
-<pinref part="S2" gate="G$1" pin="COM"/>
-</segment>
 <segment>
 <pinref part="IC2" gate="A" pin="VSB"/>
@@
 </segment>
 </net>
+<net name="N$10" class="0">
+<segment>
+<pinref part="S2" gate="G$1" pin="COM"/>
+<pinref part="IC4" gate="A" pin="VI"/>
+<wire x1="58.42" y1="10.16" x2="60.96" y2="10.16" width="0.1524" layer="91"/>
+<pinref part="C11" gate="G$1" pin="1"/>
+<wire x1="60.96" y1="10.16" x2="63.5" y2="10.16" width="0.1524" layer="91"/>
+<wire x1="60.96" y1="10.16" x2="60.96" y2="8.89" width="0.1524" layer="91"/>
+<junction x="60.96" y="10.16"/>
+</segment>
+</net>

Commit message: common
Parts:
- added C14, C15: 100u, rcl:CPOL-EUUD-6,3X8,8
- added C16: 100n, rcl:C-EUC1206
- C1: value 10u -> 100u; device rcl:CPOL-EUSMCD -> rcl:CPOL-EUUD-6,3X8,8
- C10, C9: value 22p -> 100n
- C12, C13: value 100n -> 22p
- C5: device rcl:CPOL-EUSMCD -> rcl:CPOL-EUUD-6,3X8,8
- IC4: device linear:LM340MP-05 -> linear:LM340H-05
- JP7: value 3S/4S -> 3S
- R10, R12, R14, R4, R6, R8: value 220 -> 120
- R20: value 220 -> 470
- X1: value MINI-USB-SCHIELD-32005-201 -> MINI-USB-SCHIELD-32005-301; device con-cypressindustries:MINI-USB-SCHIELD-32005-201 -> con-cypressindustries:MINI-USB-SCHIELD-32005-301
Connections:
- new net V+: X1G$1.1
- net !RESET: now also C16.1, IC3IO.PC6; no longer C13.1, IC3.PC6
- net !SS: now also IC3IO.PB2; no longer IC3.PB2
- net ADC0: now also IC3IO.PC0; no longer IC3.PC0
- net ADC1: now also IC3IO.PC1; no longer IC3.PC1
- net ADC2: now also IC3IO.PC2; no longer IC3.PC2
- net ADC3: now also IC3IO.PC3; no longer IC3.PC3
- net ADC6: now also IC3IO.ADC6; no longer IC3.ADC6
- net ADC7: now also IC3IO.ADC7; no longer IC3.ADC7
- net DIRA: now also IC3IO.PD4; no longer IC3.PD4
- net DIRB: now also IC3IO.PD7; no longer IC3.PD7
- net GND: now also C10.2, C12.1, C13.1, C14.-, C15.-, C16.2, C9.2, IC3PWR.GND; no longer C10.1, C12.2, C13.2, C9.1, IC3.GND
- net INT0: now also IC3IO.PD2; no longer IC3.PD2
- net INT1: now also IC3IO.PD3; no longer IC3.PD3
- net LED: now also IC3IO.PB0; no longer IC3.PB0
- net MISO: now also IC3IO.PB4; no longer IC3.PB4
- net MOSI: now also IC3IO.PB3; no longer IC3.PB3
- net N$10: now also C14.+; no longer C11.1
- net OC0A: now also IC3IO.PD6; no longer IC3.PD6
- net OC0B: now also IC3IO.PD5; no longer IC3.PD5
- net RX: now also IC3IO.PD0; no longer IC3.PD0
- net SCK: now also IC3IO.PB5; no longer IC3.PB5
- net SCL: now also IC3IO.PC5; no longer IC3.PC5
- net SDA: now also IC3IO.PC4; no longer IC3.PC4
- net TX: now also IC3IO.PD1; no longer IC3.PD1
- net USR: now also IC3IO.PB1; no longer IC3.PB1
- net VCC: now also C10.1, C11.1, C15.+, C9.1, IC3PWR.VCC; no longer C12.1, IC3.AREF, IC3.AVCC, IC3.VCC
- net VUSB: no longer X1G$1.1
- net XTAL1: now also C12.2, IC3IO.PB6; no longer C9.2, IC3.PB6
- net XTAL2: now also C13.2, IC3IO.PB7; no longer C10.2, IC3.PB7
Other:
- note added: "Connectors"
- note added: "Controll Unit"
- moved on the sheet: C10, C11, C12, C13, C9, J1, J2

Commit message: common
Parts:
- added LED9: Orange, led:LEDSML1206
- JP2: device pinhead:PINHD-1X6/90 -> pinhead:PINHD-1X6
- LED2: value White -> Purple
- LED8: value Orange -> White
- R2: value 1k -> 680
Connections:
- removed net !SS: IC3IO.PB2
- removed net LED: IC3IO.PB0, LED1.C
- removed net V+: X1G$1.1
- new net LEDA: IC3IO.PB1, LED2.C
- new net LEDB: IC3IO.PB2, LED1.C
- new net N$13: LED2.A, R2.1
- net ADC0: now also J2.4; no longer J2.2
- net ADC1: now also J2.5; no longer J2.3
- net ADC2: now also J2.6; no longer J2.4
- net ADC6: now also J2.2; no longer J2.8
- net ADC7: now also J2.3; no longer J2.9
- net F_ADC0: now also J1.7; no longer J1.2
- net F_ADC1: now also J1.6; no longer J1.3
- net F_ADC2: now also J1.5; no longer J1.4
- net F_ADC3: now also J1.4; no longer J1.7
- net F_ADC6: now also J1.9; no longer J1.8
- net F_ADC7: now also J1.8; no longer J1.9
- net F_GND: now also J1.1, LED8.C; no longer J1.10, LED2.C
- net F_SCL: now also J1.2; no longer J1.5
- net F_SDA: now also J1.3; no longer J1.6
- net F_VCC: now also J1.10; no longer J1.1
- net GND: now also LED9.C, S1.2; no longer LED8.C, R2.2
- net N$1: now also LED5.A; no longer LED4.A
- net N$12: now also LED6.A; no longer LED5.A
- net N$22: now also LED8.A; no longer LED7.A
- net N$30: now also LED7.A; no longer LED6.A
- net N$36: now also LED9.A; no longer LED8.A
- net N$43: now also LED4.A; no longer LED3.A
- net N$47: now also LED3.A; no longer LED2.A
- net SCL: now also J2.9; no longer J2.5
- net SDA: now also J2.8; no longer J2.6
- net USR: now also IC3IO.PB0; no longer IC3IO.PB1, R2.1
- net VCC: now also R2.2; no longer S1.2
- net VUSB: now also X1G$1.1
Other:
- note added: "LEDs and Button"
- note removed: "LED and Button"
- moved on the sheet: J1, J2, LED1, LED2, LED3, LED4, LED5, LED6, LED7, LED8, R1, R2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

Commit message: common
Parts:
- removed ZH1: LM, jst:B5B-ZR
- removed ZH2: RM, jst:B5B-ZR
- added PH1: LM, SparkFun-Connectors:CONN_05JST-VERT
- added PH2: RM, SparkFun-Connectors:CONN_05JST-VERT
Connections:
- net GND: now also PH1.3, PH2.3; no longer ZH1.3, ZH2.3
- net INT0: now also PH1.2; no longer ZH1.2
- net INT1: now also PH2.2; no longer ZH2.2
- net OUT1A: now also PH1.1; no longer ZH1.1
- net OUT1B: now also PH2.1; no longer ZH2.1
- net OUT2A: now also PH1.5; no longer ZH1.5
- net OUT2B: now also PH2.5; no longer ZH2.5
- net VCC: now also PH1.4, PH2.4; no longer ZH1.4, ZH2.4

Commit message: common
Other:
- moved on the sheet: PH2
Changed lines of the file:
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@@
 <?xml version="1.0" encoding="utf-8"?>
 <!DOCTYPE eagle SYSTEM "eagle.dtd">
-<eagle version="9.4.0">
+<eagle version="9.5.0">
 <drawing>
 <settings>
@@
 <setting verticaltext="up"/>
 </settings>
-<grid distance="0.05" unitdist="inch" unit="inch" style="dots" multiple="2" display="yes" altdistance="0.01" altunitdist="inch" altunit="inch"/>
+<grid distance="0.1" unitdist="inch" unit="inch" style="lines" multiple="1" display="no" altdistance="0.01" altunitdist="inch" altunit="inch"/>
 <layers>
 <layer number="1" name="Top" color="4" fill="1" visible="no" active="no"/>
@@
 <attribute name="VALUE" x="-8.89" y="132.08" size="1.778" layer="96" align="center"/>
 </instance>
-<instance part="PH2" gate="G$1" x="43.18" y="124.46" smashed="yes" rot="MR90">
-<attribute name="NAME" x="48.26" y="121.158" size="1.27" layer="95" rot="MR180"/>
-<attribute name="VALUE" x="35.56" y="121.158" size="1.27" layer="96" rot="MR180"/>
+<instance part="PH2" gate="G$1" x="43.18" y="125.73" smashed="yes" rot="MR90">
+<attribute name="NAME" x="48.26" y="122.428" size="1.27" layer="95" rot="MR180"/>
+<attribute name="VALUE" x="35.56" y="122.428" size="1.27" layer="96" rot="MR180"/>
 </instance>
 <instance part="PH1" gate="G$1" x="12.7" y="125.73" smashed="yes" rot="MR90">
@@
 <pinref part="PH2" gate="G$1" pin="3"/>
 <wire x1="27.94" y1="134.62" x2="43.18" y2="134.62" width="0.1524" layer="91"/>
-<wire x1="43.18" y1="134.62" x2="43.18" y2="132.08" width="0.1524" layer="91"/>
+<wire x1="43.18" y1="134.62" x2="43.18" y2="133.35" width="0.1524" layer="91"/>
 <wire x1="27.94" y1="134.62" x2="27.94" y2="132.08" width="0.1524" layer="91"/>
 <junction x="27.94" y="134.62"/>
@@
 <pinref part="PH2" gate="G$1" pin="4"/>
 <wire x1="27.94" y1="137.16" x2="45.72" y2="137.16" width="0.1524" layer="91"/>
-<wire x1="45.72" y1="137.16" x2="45.72" y2="132.08" width="0.1524" layer="91"/>
+<wire x1="45.72" y1="137.16" x2="45.72" y2="133.35" width="0.1524" layer="91"/>
 <wire x1="27.94" y1="137.16" x2="27.94" y2="139.7" width="0.1524" layer="91"/>
 <junction x="27.94" y="137.16"/>
@@
 <segment>
 <pinref part="PH2" gate="G$1" pin="2"/>
-<wire x1="40.64" y1="132.08" x2="40.64" y2="144.78" width="0.1524" layer="91"/>
+<wire x1="40.64" y1="133.35" x2="40.64" y2="144.78" width="0.1524" layer="91"/>
 <wire x1="38.1" y1="147.32" x2="40.64" y2="144.78" width="0.1524" layer="91"/>
 <label x="40.64" y="144.78" size="1.778" layer="95" rot="MR270"/>
@@
 <wire x1="45.72" y1="147.32" x2="48.26" y2="144.78" width="0.1524" layer="91"/>
 <pinref part="PH2" gate="G$1" pin="5"/>
-<wire x1="48.26" y1="144.78" x2="48.26" y2="132.08" width="0.1524" layer="91"/>
+<wire x1="48.26" y1="144.78" x2="48.26" y2="133.35" width="0.1524" layer="91"/>
 <label x="48.26" y="144.78" size="1.778" layer="95" rot="MR270"/>
 </segment>
@@
 <segment>
 <wire x1="35.56" y1="147.32" x2="38.1" y2="144.78" width="0.1524" layer="91"/>
-<wire x1="38.1" y1="144.78" x2="38.1" y2="132.08" width="0.1524" layer="91"/>
+<wire x1="38.1" y1="144.78" x2="38.1" y2="133.35" width="0.1524" layer="91"/>
 <pinref part="PH2" gate="G$1" pin="1"/>
 <label x="38.1" y="144.78" size="1.778" layer="95" rot="MR270"/>
